File: layouts/lsm6dsl/lsm6dsl.kicad_pcb (KiCad board)
At the start: 2 copper layers, 2 parts

Commit message: ready to order i think
Connections:
- net VCC renamed VDDIO
Changed lines of the file:
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@@
     (net 6 "ic.footprint.pins[1].net-net")
     (net 7 "gnd")
-    (net 8 "VCC")
+    (net 8 "VDDIO")
     (footprint "atopile:LGA-14_L3.0-W2.5-P0.50-TL-eab322"
         (layer "F.Cu")
@@
             (size 0.28 0.68)
             (layers "F.Cu" "F.Mask" "F.Paste")
-            (net 8 "VCC")
+            (net 8 "VDDIO")
         )
         (pad "6" smd rect
@@
             (size 0.68 0.28)
             (layers "F.Cu" "F.Mask" "F.Paste")
-            (net 8 "VCC")
+            (net 8 "VDDIO")
         )
         (pad "9" smd rect
@@
             (size 0.28 0.68)
             (layers "F.Cu" "F.Mask" "F.Paste")
-            (net 8 "VCC")
+            (net 8 "VDDIO")
         )
         (pad "13" smd rect
@@
             (size 0.79 0.54)
             (layers "F.Cu" "F.Mask" "F.Paste")
-            (net 8 "VCC")
+            (net 8 "VDDIO")
         )
         (pad "2" smd rect

Commit message: updates
Connections:
- net VDDIO renamed VCC
Changed lines of the file:
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@@
     (net 6 "ic.footprint.pins[1].net-net")
     (net 7 "gnd")
-    (net 8 "VDDIO")
+    (net 8 "VCC")
     (footprint "atopile:LGA-14_L3.0-W2.5-P0.50-TL-eab322"
         (layer "F.Cu")
@@
             (size 0.28 0.68)
             (layers "F.Cu" "F.Mask" "F.Paste")
-            (net 8 "VDDIO")
+            (net 8 "VCC")
         )
         (pad "6" smd rect
@@
             (size 0.68 0.28)
             (layers "F.Cu" "F.Mask" "F.Paste")
-            (net 8 "VDDIO")
+            (net 8 "VCC")
         )
         (pad "9" smd rect
@@
             (size 0.28 0.68)
             (layers "F.Cu" "F.Mask" "F.Paste")
-            (net 8 "VDDIO")
+            (net 8 "VCC")
         )
         (pad "13" smd rect
@@
             (size 0.79 0.54)
             (layers "F.Cu" "F.Mask" "F.Paste")
-            (net 8 "VDDIO")
+            (net 8 "VCC")
         )
         (pad "2" smd rect
