File: layouts/default/default.kicad_pcb (KiCad board)
At the start: 4 copper layers, 27.5 x 14.2 mm, 21 parts

Commit message: ready to order i think
Parts:
- added R6: 10kΩ ±1% 50mW, atopile:R0201-27027e, B.Cu at (79.1, 59.4)
Connections:
- C1 pad 1: hv -> hv-1
- C2 pad 1: hv-1 -> hv-2
- C3 pad 1: hv-2 -> hv
- C4 pad 1: hv-1 -> hv-2
- C5 pad 1: hv-2 -> hv
- C6 pad 1: hv-2 -> hv
- C7 pad 1: hv-2 -> hv
- C8 pad 1: hv-2 -> hv
- C9 pad 1: hv-2 -> hv
- L1 pad 18: uc-line-1 -> uc-line-9
- L1 pad 22: uc-line-7 -> EN
- L1 pad 23: uc-line-3 -> uc-line
- L1 pad 24: uc-line-6 -> uc-line-2
- L1 pad 26: uc-line-9 -> uc-line-10
- L1 pad 27: uc-line-4 -> uc-line-8
- L1 pad 28: uc-line -> uc-line-7
- L1 pad 29: uc-line-2 -> uc-line-6
- L1 pad 3: hv-2 -> hv
- L1 pad 30: line-1 -> line
- L1 pad 31: line -> line-1
- L1 pad 5: uc-line-8 -> uc-line-3
- L1 pad 6: uc-line-10 -> uc-line-4
- L1 pad 8: EN -> uc-line-1
- L2 pad 2: hv-2 -> hv
- MIC1 pad 5: hv-2 -> hv
- R5 pad 1: hv-2 -> hv
- U1 pad A4: hv -> hv-1
- U1 pad A6: line -> line-1
- U1 pad A7: line-1 -> line
- U1 pad A9: hv -> hv-1
- U1 pad B4: hv -> hv-1
- U1 pad B6: line -> line-1
- U1 pad B7: line-1 -> line
- U1 pad B9: hv -> hv-1
- U2 pad 1: hv -> hv-1
- U2 pad 10: hv-1 -> hv-2
- U2 pad 7: hv -> hv-1
- U3 pad 4: hv-1 -> hv-2
- U4 pad 12: hv-2 -> hv
- U4 pad 5: hv-2 -> hv
- U4 pad 8: hv-2 -> hv
Routing:
- net hv: track 24.2 -> 35.5 mm, vias 3 -> 2
- net hv-2: track 32.9 -> 23.2 mm
- net EN: track 3.17 -> 12.6 mm, vias 0 -> 1
- net hv-1: track 22.4 -> 24.5 mm, vias 2 -> 3
- net gnd: track 67.5 -> 68.3 mm, vias 15 -> 13
- net line: track 19.4 -> 20.1 mm
- net line-1: track 19.5 -> 20.0 mm
- net uc.footprint.pins[12].net-net: vias 1 -> 0
